File: electrical/Particulate_matter_sensor/Particulate_matter_sensor.kicad_sch (KiCad schematic)
At the start: 4 parts, among them J1 c8-inlet, U1 ESP32-C3_SUPERMINI, U2 BOB-12009

Commit message: updates
Parts:
- added GND, POS5: TestPoint, TestPoint:TestPoint_Pad_D2.0mm, symbol Connector:TestPoint
- added PM10_N3_PWM: ~, symbol laser_sensor:LaserParticulateSensor
- added POS3P3: TestPoint, symbol Connector:TestPoint
- added TFT_LCD: Conn_01x04_Socket, symbol Connector:Conn_01x04_Socket
Connections:
- net RX/PWM: now reaches U1.20 (GPIO20)
- net RX/PWM: now also PM10_N3_PWM.4 (PWM)
- net TX: now reaches U1.21 (GPIO21)
- net TX: now also PM10_N3_PWM.3 (RXD)
- net +3.3V: now reaches U1.3.3 (3V3)
- net +3.3V: now also POS3P3.1, TFT_LCD.3 (Pin_3)
- net +5V: now reaches U1.5V
- net +5V: now also PS1.4 (+Vout), PM10_N3_PWM.2 (VCC), POS5.1
- net I2C_SDA: now reaches U1.8 (GPIO8)
- net I2C_SDA: now also TFT_LCD.1 (Pin_1)
- net I2C_SCL: now reaches U1.9 (GPIO9)
- net I2C_SCL: now also TFT_LCD.2 (Pin_2)
- net GND: now reaches U1.G (GND)
- net GND: now also PS1.3 (-Vout), U2.GND_1 (GND), U2.GND_2 (GND), GND.1, PM10_N3_PWM.1 (GND), TFT_LCD.4 (Pin_4)
- net at PS1.1 (AC/L): now also J1.1 (N)
- net at PS1.2 (AC/N): now also J1.2 (L)
Other:
- moved on the sheet: J1
